File: Electronic Board/Kicad Project/SailboatMainBoard.kicad_pcb (KiCad board)
At the start: 2 copper layers, 85.7 x 104.1 mm, 63 parts, among them J1 Conn_01x02, J10 Conn_01x02, J11 Conn_01x03_Male, J12 Conn_01x03_Male, J13 Conn_01x03_Male, J14 Conn_01x03_Male, J15 Conn_01x04, J16 Conn_01x04, J17 Conn_01x04, J18 Conn_01x04, J19 Conn_01x03, J2 Conn_01x08, J20 Conn_01x03, J21 Conn_01x02, J22 Conn_01x02, J23 Conn_02x20_Odd_Even, J24 Conn_01x03, J25 Conn_01x03_Female, J26 Conn_01x03_Female, J27 Conn_01x03_Female, J28 Conn_01x03_Female, J29 Conn_01x03_Female, J3 Conn_01x08, J30 Conn_01x03_Female, J31 Conn_01x04, J32 Conn_01x04, J33 Conn_01x08_Female, J34 Conn_01x02, J35 Conn_01x02, J36 Conn_01x02, J37 Conn_01x02, J4 Conn_01x08, J5 Conn_02x18_Odd_Even, J6 Conn_01x08, J7 Conn_01x08, J8 Conn_01x08, J9 Conn_01x02, U1 L7805, U2 L7805, U3 L7805

Commit message: Finished board-v0.1
Parts:
- moved REF** 1.27 mm to (177.2, 54.6)
Changed lines of the file:
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@@
     (links 129)
     (no_connects 0)
-    (area 102.184999 53.289999 188.010001 157.530001)
+    (area 95.915 36.094999 192.278572 164.535)
     (thickness 1.6)
     (drawings 48)
@@
   )
   (setup
-    (last_trace_width 0.5)
+    (last_trace_width 0.25)
     (user_trace_width 0.5)
     (trace_clearance 0.2)
@@
   )
   (module Mounting_Holes:MountingHole_2.5mm (layer F.Cu)
-    (at 177.165 55.88)
+    (at 177.165 54.61)
     (descr "Mounting Hole 2.5mm, no annular")
     (tags "mounting hole 2.5mm no annular")
@@
   (gr_circle (center 184.15 118.11) (end 181.61 118.11) (layer Eco1.User) (width 0.2))
   (gr_circle (center 135.255 118.11) (end 132.715 118.11) (layer Eco1.User) (width 0.2))
-  (gr_circle (center 177.165 55.88) (end 179.07 55.88) (layer Eco2.User) (width 0.2))
+  (gr_circle (center 177.165 54.61) (end 179.07 54.61) (layer Eco2.User) (width 0.2))
   (gr_circle (center 128.905 55.88) (end 130.81 55.88) (layer Eco2.User) (width 0.2))
   (gr_circle (center 177.165 137.16) (end 179.07 137.16) (layer Eco2.User) (width 0.2))
