File: Electronic Board/Sailboat Kicad/Board1-Arduino/Connectors.sch (KiCad schematic (older format))
At the start: 33 parts, among them J1 Conn_01x02, J10 Conn_01x02, J11 Conn_01x03_Male, J12 Conn_01x03_Male, J13 Conn_01x03_Male, J14 Conn_01x03_Male, J15 Conn_01x04, J16 Conn_01x04, J17 Conn_01x04, J18 Conn_01x04, J19 Conn_01x03, J20 Conn_01x03, J21 Conn_01x02, J22 Conn_01x02, J23 Conn_01x06, J24 Conn_01x03, J25 Conn_01x06, J26 Conn_02x02_Odd_Even, J31 Conn_01x04, J32 Conn_01x04, J34 Conn_01x02, J35 Conn_01x02, J36 Conn_01x02, J37 Conn_01x02, J9 Conn_01x02

Commit message: Finished board-v0.1
Parts:
- removed R10, R11, R2, R4, R6, R7, R8, R9: 4k7, Resistors_THT:R_Axial_DIN0204_L3.6mm_D1.6mm_P5.08mm_Horizontal, symbol R_Small
Changed lines of the file:
@@
 Wire Wire Line
 	1900 5150 2000 5150
-$Comp
-L R_Small R2
-U 1 1 5A965541
-P 2100 4450
-F 0 "R2" H 2130 4470 50  0000 L CNN
-F 1 "4k7" H 1900 4400 50  0000 L CNN
-F 2 "Resistors_THT:R_Axial_DIN0204_L3.6mm_D1.6mm_P5.08mm_Horizontal" H 2100 4450 50  0001 C CNN
-F 3 "" H 2100 4450 50  0001 C CNN
-	1    2100 4450
-	1    0    0    -1
-$EndComp
-$Comp
-L R_Small R6
-U 1 1 5A9655AD
-P 2200 4650
-F 0 "R6" H 2230 4670 50  0000 L CNN
-F 1 "4k7" H 2230 4610 50  0000 L CNN
-F 2 "Resistors_THT:R_Axial_DIN0204_L3.6mm_D1.6mm_P5.08mm_Horizontal" H 2200 4650 50  0001 C CNN
-F 3 "" H 2200 4650 50  0001 C CNN
-	1    2200 4650
-	1    0    0    -1
-$EndComp
-Wire Wire Line
-	2200 4750 2200 4950
-Connection ~ 2200 4950
-Wire Wire Line
-	2100 4550 2100 4850
-Connection ~ 2100 4850
 Text HLabel 2000 5050 2    60   BiDi ~ 0
 5V-Sensors
-Text HLabel 2200 4250 2    60   BiDi ~ 0
-5V-Sensors
-Wire Wire Line
-	2100 4350 2100 4250
-Wire Wire Line
-	2100 4250 2200 4250
-Wire Wire Line
-	2200 4250 2200 4550
 $Comp
 L Conn_01x04 J17
@@
 Wire Wire Line
 	3400 5150 3500 5150
-$Comp
-L R_Small R8
-U 1 1 5A965B96
-P 3600 4450
-F 0 "R8" H 3630 4470 50  0000 L CNN
-F 1 "4k7" H 3400 4400 50  0000 L CNN
-F 2 "Resistors_THT:R_Axial_DIN0204_L3.6mm_D1.6mm_P5.08mm_Horizontal" H 3600 4450 50  0001 C CNN
-F 3 "" H 3600 4450 50  0001 C CNN
-	1    3600 4450
-	1    0    0    -1
-$EndComp
-$Comp
-L R_Small R10
-U 1 1 5A965B9C
-P 3700 4650
-F 0 "R10" H 3730 4670 50  0000 L CNN
-F 1 "4k7" H 3730 4610 50  0000 L CNN
-F 2 "Resistors_THT:R_Axial_DIN0204_L3.6mm_D1.6mm_P5.08mm_Horizontal" H 3700 4650 50  0001 C CNN
-F 3 "" H 3700 4650 50  0001 C CNN
-	1    3700 4650
-	1    0    0    -1
-$EndComp
-Wire Wire Line
-	3700 4750 3700 4950
-Connection ~ 3700 4950
-Wire Wire Line
-	3600 4550 3600 4850
-Connection ~ 3600 4850
 Text HLabel 3500 5050 2    60   BiDi ~ 0
 5V-Sensors
-Text HLabel 3700 4250 2    60   BiDi ~ 0
-5V-Sensors
-Wire Wire Line
-	3600 4350 3600 4250
-Wire Wire Line
-	3600 4250 3700 4250
-Wire Wire Line
-	3700 4250 3700 4550
 $Comp
 L Conn_01x04 J16
@@
 Wire Wire Line
 	1900 6300 2000 6300
-$Comp
-L R_Small R4
-U 1 1 5A965E1F
-P 2100 5600
-F 0 "R4" H 2130 5620 50  0000 L CNN
-F 1 "4k7" H 1900 5550 50  0000 L CNN
-F 2 "Resistors_THT:R_Axial_DIN0204_L3.6mm_D1.6mm_P5.08mm_Horizontal" H 2100 5600 50  0001 C CNN
-F 3 "" H 2100 5600 50  0001 C CNN
-	1    2100 5600
-	1    0    0    -1
-$EndComp
-$Comp
-L R_Small R7
-U 1 1 5A965E25
-P 2200 5800
-F 0 "R7" H 2230 5820 50  0000 L CNN
-F 1 "4k7" H 2230 5760 50  0000 L CNN
-F 2 "Resistors_THT:R_Axial_DIN0204_L3.6mm_D1.6mm_P5.08mm_Horizontal" H 2200 5800 50  0001 C CNN
-F 3 "" H 2200 5800 50  0001 C CNN
-	1    2200 5800
-	1    0    0    -1
-$EndComp
-Wire Wire Line
-	2200 5900 2200 6100
-Connection ~ 2200 6100
-Wire Wire Line
-	2100 5700 2100 6000
-Connection ~ 2100 6000
 Text HLabel 2000 6200 2    60   BiDi ~ 0
 5V-Sensors
-Text HLabel 2200 5400 2    60   BiDi ~ 0
-5V-Sensors
-Wire Wire Line
-	2100 5500 2100 5400
-Wire Wire Line
-	2100 5400 2200 5400
-Wire Wire Line
-	2200 5400 2200 5700
 $Comp
 L Conn_01x04 J18
@@
 Wire Wire Line
 	3400 6300 3500 6300
-$Comp
-L R_Small R9
-U 1 1 5A965E46
-P 3600 5600
-F 0 "R9" H 3630 5620 50  0000 L CNN
-F 1 "4k7" H 3400 5550 50  0000 L CNN
-F 2 "Resistors_THT:R_Axial_DIN0204_L3.6mm_D1.6mm_P5.08mm_Horizontal" H 3600 5600 50  0001 C CNN
-F 3 "" H 3600 5600 50  0001 C CNN
-	1    3600 5600
-	1    0    0    -1
-$EndComp
-$Comp
-L R_Small R11
-U 1 1 5A965E4C
-P 3700 5800
-F 0 "R11" H 3730 5820 50  0000 L CNN
-F 1 "4k7" H 3730 5760 50  0000 L CNN
-F 2 "Resistors_THT:R_Axial_DIN0204_L3.6mm_D1.6mm_P5.08mm_Horizontal" H 3700 5800 50  0001 C CNN
-F 3 "" H 3700 5800 50  0001 C CNN
-	1    3700 5800
-	1    0    0    -1
-$EndComp
-Wire Wire Line
-	3700 5900 3700 6100
-Connection ~ 3700 6100
-Wire Wire Line
-	3600 5700 3600 6000
-Connection ~ 3600 6000
 Text HLabel 3500 6200 2    60   BiDi ~ 0
 5V-Sensors
-Text HLabel 3700 5400 2    60   BiDi ~ 0
-5V-Sensors
-Wire Wire Line
-	3600 5500 3600 5400
-Wire Wire Line
-	3600 5400 3700 5400
-Wire Wire Line
-	3700 5400 3700 5700
 Wire Notes Line
 	1000 4100 4450 4100

Commit message: Cleaned up, and added security, text and better usability, preparation for board v2
Parts:
- added D4, D5: D_Schottky, Diodes_THT:D_5W_P10.16mm_Horizontal, symbol D_Schottky
Connections:
- net 5V-Sensors: now also J15.1 (Pin_1), J16.1 (Pin_1), J17.1 (Pin_1), J18.1 (Pin_1); no longer J15.2 (Pin_2), J16.2 (Pin_2), J17.2 (Pin_2), J18.2 (Pin_2)
- net BAT+: now also D4.2 (A), D5.2 (A); no longer J10.2 (Pin_2), J9.2 (Pin_2)
- net GND: now also J15.2 (Pin_2), J16.2 (Pin_2), J17.2 (Pin_2), J18.2 (Pin_2); no longer J15.1 (Pin_1), J16.1 (Pin_1), J17.1 (Pin_1), J18.1 (Pin_1)
- new net: D4.1 (K), J9.2 (Pin_2)
- new net: D5.1 (K), J10.2 (Pin_2)
Other:
- moved on the sheet: J10, J9
Changed lines of the file:
@@
 L Conn_01x02 J9
 U 1 1 5A95F23C
-P 1800 1550
-F 0 "J9" H 1800 1650 50  0000 C CNN
-F 1 "Conn_01x02" H 1800 1350 50  0000 C CNN
-F 2 "Sailboat:BAT-CONN" H 1800 1550 50  0001 C CNN
-F 3 "" H 1800 1550 50  0001 C CNN
-	1    1800 1550
-	-1   0    0    1
-$EndComp
-Text HLabel 2100 1450 2    60   BiDi ~ 0
+P 1800 1800
+F 0 "J9" H 1800 1900 50  0000 C CNN
+F 1 "Conn_01x02" H 1800 1600 50  0000 C CNN
+F 2 "Sailboat:BAT-CONN" H 1800 1800 50  0001 C CNN
+F 3 "" H 1800 1800 50  0001 C CNN
+	1    1800 1800
+	-1   0    0    1
+$EndComp
+Text HLabel 2400 1700 2    60   BiDi ~ 0
 BAT+
-Text HLabel 2100 1550 2    60   BiDi ~ 0
+Text HLabel 2100 1800 2    60   BiDi ~ 0
 BAT-
 Wire Wire Line
-	2100 1450 2000 1450
-Wire Wire Line
-	2100 1550 2000 1550
+	2100 1700 2000 1700
+Wire Wire Line
+	2100 1800 2000 1800
 $Comp
 L Conn_01x02 J10
 U 1 1 5A95F2D2
-P 1800 1950
-F 0 "J10" H 1800 2050 50  0000 C CNN
-F 1 "Conn_01x02" H 1800 1750 50  0000 C CNN
-F 2 "Sailboat:BAT-CONN" H 1800 1950 50  0001 C CNN
-F 3 "" H 1800 1950 50  0001 C CNN
-	1    1800 1950
-	-1   0    0    1
-$EndComp
-Text HLabel 2100 1850 2    60   BiDi ~ 0
+P 1800 2200
+F 0 "J10" H 1800 2300 50  0000 C CNN
+F 1 "Conn_01x02" H 1800 2000 50  0000 C CNN
+F 2 "Sailboat:BAT-CONN" H 1800 2200 50  0001 C CNN
+F 3 "" H 1800 2200 50  0001 C CNN
+	1    1800 2200
+	-1   0    0    1
+$EndComp
+Text HLabel 2400 2100 2    60   BiDi ~ 0
 BAT+
-Text HLabel 2100 1950 2    60   BiDi ~ 0
+Text HLabel 2100 2200 2    60   BiDi ~ 0
 BAT-
 Wire Wire Line
-	2100 1850 2000 1850
-Wire Wire Line
-	2100 1950 2000 1950
+	2100 2100 2000 2100
+Wire Wire Line
+	2100 2200 2000 2200
 Text HLabel 2000 2750 2    60   Input ~ 0
 Servo-Sail
@@
 	1900 2950 2000 2950
 $Comp
-L GND #PWR07
+L GND #PWR08
 U 1 1 5A95F4EF
 P 2000 2950
-F 0 "#PWR07" H 2000 2700 50  0001 C CNN
+F 0 "#PWR08" H 2000 2700 50  0001 C CNN
 F 1 "GND" H 2000 2800 50  0000 C CNN
 F 2 "" H 2000 2950 50  0001 C CNN
@@
 	1900 3500 2000 3500
 $Comp
-L GND #PWR08
+L GND #PWR09
 U 1 1 5A95F560
 P 2000 3500
-F 0 "#PWR08" H 2000 3250 50  0001 C CNN
+F 0 "#PWR09" H 2000 3250 50  0001 C CNN
 F 1 "GND" H 2000 3350 50  0000 C CNN
 F 2 "" H 2000 3500 50  0001 C CNN
@@
 	3450 2950 3550 2950
 $Comp
-L GND #PWR09
+L GND #PWR010
 U 1 1 5A95F5D9
 P 3550 2950
-F 0 "#PWR09" H 3550 2700 50  0001 C CNN
+F 0 "#PWR010" H 3550 2700 50  0001 C CNN
 F 1 "GND" H 3550 2800 50  0000 C CNN
 F 2 "" H 3550 2950 50  0001 C CNN
@@
 	3450 3500 3550 3500
 $Comp
-L GND #PWR010
+L GND #PWR011
 U 1 1 5A95F621
 P 3550 3500
-F 0 "#PWR010" H 3550 3250 50  0001 C CNN
+F 0 "#PWR011" H 3550 3250 50  0001 C CNN
 F 1 "GND" H 3550 3350 50  0000 C CNN
 F 2 "" H 3550 3500 50  0001 C CNN
@@
 Text Notes 1050 1000 0    60   ~ 0
 Battery Input
-Text Notes 1050 1550 0    60   ~ 0
+Text Notes 1050 1800 0    60   ~ 0
 Battery Output
-Text Notes 1050 1950 0    60   ~ 0
+Text Notes 1050 2200 0    60   ~ 0
 Battery Output
 Text Notes 1000 2450 0    60   ~ 0
@@
 SCL
 $Comp
-L GND #PWR011
+L GND #PWR012
 U 1 1 5A962CDB
-P 2000 5150
-F 0 "#PWR011" H 2000 4900 50  0001 C CNN
-F 1 "GND" H 2000 5000 50  0000 C CNN
-F 2 "" H 2000 5150 50  0001 C CNN
-F 3 "" H 2000 5150 50  0001 C CNN
-	1    2000 5150
+P 2000 5050
+F 0 "#PWR012" H 2000 4800 50  0001 C CNN
+F 1 "GND" H 2000 4900 50  0000 C CNN
+F 2 "" H 2000 5050 50  0001 C CNN
+F 3 "" H 2000 5050 50  0001 C CNN
+	1    2000 5050
 	0    -1   -1   0
 $EndComp
@@
 Wire Wire Line
 	1900 5150 2000 5150
-Text HLabel 2000 5050 2    60   BiDi ~ 0
+Text HLabel 2000 5150 2    60   BiDi ~ 0
 5V-Sensors
 $Comp
@@
 SCL
 $Comp
-L GND #PWR012
+L GND #PWR013
 U 1 1 5A965B8C
-P 3500 5150
-F 0 "#PWR012" H 3500 4900 50  0001 C CNN
-F 1 "GND" H 3500 5000 50  0000 C CNN
-F 2 "" H 3500 5150 50  0001 C CNN
-F 3 "" H 3500 5150 50  0001 C CNN
-	1    3500 5150
+P 3500 5050
+F 0 "#PWR013" H 3500 4800 50  0001 C CNN
+F 1 "GND" H 3500 4900 50  0000 C CNN
+F 2 "" H 3500 5050 50  0001 C CNN
+F 3 "" H 3500 5050 50  0001 C CNN
+	1    3500 5050
 	0    -1   -1   0
 $EndComp
@@
 Wire Wire Line
 	3400 5150 3500 5150
-Text HLabel 3500 5050 2    60   BiDi ~ 0
+Text HLabel 3500 5150 2    60   BiDi ~ 0
 5V-Sensors
 $Comp
@@
 SCL
 $Comp
-L GND #PWR013
+L GND #PWR014
 U 1 1 5A965E15
-P 2000 6300
-F 0 "#PWR013" H 2000 6050 50  0001 C CNN
-F 1 "GND" H 2000 6150 50  0000 C CNN
-F 2 "" H 2000 6300 50  0001 C CNN
-F 3 "" H 2000 6300 50  0001 C CNN
-	1    2000 6300
+P 2000 6200
+F 0 "#PWR014" H 2000 5950 50  0001 C CNN
+F 1 "GND" H 2000 6050 50  0000 C CNN
+F 2 "" H 2000 6200 50  0001 C CNN
+F 3 "" H 2000 6200 50  0001 C CNN
+	1    2000 6200
 	0    -1   -1   0
 $EndComp
@@
 Wire Wire Line
 	1900 6300 2000 6300
-Text HLabel 2000 6200 2    60   BiDi ~ 0
+Text HLabel 2000 6300 2    60   BiDi ~ 0
 5V-Sensors
 $Comp
@@
 SCL
 $Comp
-L GND #PWR014
+L GND #PWR015
 U 1 1 5A965E3C
-P 3500 6300
-F 0 "#PWR014" H 3500 6050 50  0001 C CNN
-F 1 "GND" H 3500 6150 50  0000 C CNN
-F 2 "" H 3500 6300 50  0001 C CNN
-F 3 "" H 3500 6300 50  0001 C CNN
-	1    3500 6300
+P 3500 6200
+F 0 "#PWR015" H 3500 5950 50  0001 C CNN
+F 1 "GND" H 3500 6050 50  0000 C CNN
+F 2 "" H 3500 6200 50  0001 C CNN
+F 3 "" H 3500 6200 50  0001 C CNN
+	1    3500 6200
 	0    -1   -1   0
 $EndComp
@@
 Wire Wire Line
 	3400 6300 3500 6300
-Text HLabel 3500 6200 2    60   BiDi ~ 0
+Text HLabel 3500 6300 2    60   BiDi ~ 0
 5V-Sensors
 Wire Notes Line
@@
 5V-Sensors
 $Comp
-L GND #PWR015
+L GND #PWR016
 U 1 1 5A9669C7
 P 5750 1100
-F 0 "#PWR015" H 5750 850 50  0001 C CNN
+F 0 "#PWR016" H 5750 850 50  0001 C CNN
 F 1 "GND" H 5750 950 50  0000 C CNN
 F 2 "" H 5750 1100 50  0001 C CNN
@@
 5V-Sensors
 $Comp
-L GND #PWR016
+L GND #PWR017
 U 1 1 5A967044
 P 5750 1650
-F 0 "#PWR016" H 5750 1400 50  0001 C CNN
+F 0 "#PWR017" H 5750 1400 50  0001 C CNN
 F 1 "GND" H 5750 1500 50  0000 C CNN
 F 2 "" H 5750 1650 50  0001 C CNN
@@
 5V-Sensors
 $Comp
-L GND #PWR017
+L GND #PWR018
 U 1 1 5A967170
 P 7050 1100
-F 0 "#PWR017" H 7050 850 50  0001 C CNN
+F 0 "#PWR018" H 7050 850 50  0001 C CNN
 F 1 "GND" H 7050 950 50  0000 C CNN
 F 2 "" H 7050 1100 50  0001 C CNN
@@
 	1000 700  3400 700
 Wire Notes Line
-	3400 700  3400 2100
-Wire Notes Line
-	3400 2100 1000 2100
-Wire Notes Line
-	1000 2100 1000 700
+	3400 700  3400 2350
+Wire Notes Line
+	1000 700  1000 2350
 Text Notes 1050 650  0    60   ~ 0
 Battery
@@
 D0
 $Comp
-L GND #PWR018
+L GND #PWR019
 U 1 1 5A967B3C
 P 5750 2800
-F 0 "#PWR018" H 5750 2550 50  0001 C CNN
+F 0 "#PWR019" H 5750 2550 50  0001 C CNN
 F 1 "GND" H 5750 2650 50  0000 C CNN
 F 2 "" H 5750 2800 50  0001 C CNN
@@
 D1
 $Comp
-L GND #PWR019
+L GND #PWR020
 U 1 1 5A967DD0
 P 5750 3200
-F 0 "#PWR019" H 5750 2950 50  0001 C CNN
+F 0 "#PWR020" H 5750 2950 50  0001 C CNN
 F 1 "GND" H 5750 3050 50  0000 C CNN
 F 2 "" H 5750 3200 50  0001 C CNN
@@
 $EndComp
 $Comp
-L GND #PWR020
+L GND #PWR021
 U 1 1 5A9A9197
 P 7200 2950
-F 0 "#PWR020" H 7200 2700 50  0001 C CNN
+F 0 "#PWR021" H 7200 2700 50  0001 C CNN
 F 1 "GND" H 7200 2800 50  0000 C CNN
 F 2 "" H 7200 2950 50  0001 C CNN
@@
 $EndComp
 $Comp
-L GND #PWR021
+L GND #PWR022
 U 1 1 5A9A98D8
 P 8550 2950
-F 0 "#PWR021" H 8550 2700 50  0001 C CNN
+F 0 "#PWR022" H 8550 2700 50  0001 C CNN
 F 1 "GND" H 8550 2800 50  0000 C CNN
 F 2 "" H 8550 2950 50  0001 C CNN
@@
 5V-Rpi
 $Comp
-L GND #PWR022
+L GND #PWR023
 U 1 1 5AB2AB72
 P 6650 4400
-F 0 "#PWR022" H 6650 4150 50  0001 C CNN
+F 0 "#PWR023" H 6650 4150 50  0001 C CNN
 F 1 "GND" H 6650 4250 50  0000 C CNN
 F 2 "" H 6650 4400 50  0001 C CNN
@@
 $EndComp
 $Comp
-L GND #PWR023
+L GND #PWR024
 U 1 1 5AB2AD8D
 P 6650 4500
-F 0 "#PWR023" H 6650 4250 50  0001 C CNN
+F 0 "#PWR024" H 6650 4250 50  0001 C CNN
 F 1 "GND" H 6650 4350 50  0000 C CNN
 F 2 "" H 6650 4500 50  0001 C CNN
@@
 	6650 4500 6750 4500
 NoConn ~ 5400 5200
+$Comp
+L D_Schottky D4
+U 1 1 5B0DC780
+P 2250 1700
+F 0 "D4" H 2250 1800 50  0000 C CNN
+F 1 "D_Schottky" H 2250 1600 50  0000 C CNN
+F 2 "Diodes_THT:D_5W_P10.16mm_Horizontal" H 2250 1700 50  0001 C CNN
+F 3 "" H 2250 1700 50  0001 C CNN
+	1    2250 1700
+	1    0    0    -1
+$EndComp
+Wire Notes Line
+	1000 2350 3400 2350
+$Comp
+L D_Schottky D5
+U 1 1 5B0DCBC5
+P 2250 2100
+F 0 "D5" H 2250 2200 50  0000 C CNN
+F 1 "D_Schottky" H 2250 2000 50  0000 C CNN
+F 2 "Diodes_THT:D_5W_P10.16mm_Horizontal" H 2250 2100 50  0001 C CNN
+F 3 "" H 2250 2100 50  0001 C CNN
+	1    2250 2100
+	1    0    0    -1
+$EndComp
 $EndSCHEMATC

Commit message: Updated version of Kicad, rendered images and BOM
Parts:
- removed J1, J10, J9: Conn_01x02, Sailboat:BAT-CONN, symbol Conn_01x02
- removed J11, J12, J13, J14: Conn_01x03_Male, Pin_Headers:Pin_Header_Angled_1x03_Pitch2.54mm, symbol Conn_01x03_Male
- removed J15, J16, J17, J18, J31, J32: Conn_01x04, Connectors_JST:JST_PH_S4B-PH-K_04x2.00mm_Angled, symbol Conn_01x04
- removed J19, J20, J24: Conn_01x03, Connectors_JST:JST_PH_S3B-PH-K_03x2.00mm_Angled, symbol Conn_01x03
- removed J21, J22, J34, J35: Conn_01x02, Connectors_JST:JST_PH_S2B-PH-K_02x2.00mm_Angled, symbol Conn_01x02
- removed J23, J25: Conn_01x06, Pin_Headers:Pin_Header_Straight_1x06_Pitch2.54mm, symbol Conn_01x06
- removed J26: Conn_02x02_Odd_Even, Pin_Headers:Pin_Header_Straight_2x02_Pitch2.54mm, symbol Conn_02x02_Odd_Even
- removed J36, J37: Conn_01x02, Pin_Headers:Pin_Header_Straight_1x02_Pitch2.54mm, symbol Conn_01x02
- added J1, J14, J15, J2: Conn_01x03_Male, Connector_PinHeader_2.54mm:PinHeader_1x03_P2.54mm_Horizontal, symbol Connector:Conn_01x03_Male
- added J10, J20, J21, J8: Conn_01x02_Male, Connector_JST:JST_PH_S2B-PH-K_1x02_P2.00mm_Horizontal, symbol Connector:Conn_01x02_Male
- added J11, J9: Conn_01x02_Male, Connector_PinHeader_2.54mm:PinHeader_1x02_P2.54mm_Vertical, symbol Connector:Conn_01x02_Male
- added J12, J13, J23, J25, J3, J4: Conn_01x04_Male, Connector_JST:JST_PH_S4B-PH-K_1x04_P2.00mm_Horizontal, symbol Connector:Conn_01x04_Male
- added J16, J17: Conn_01x06_Male, Connector_PinHeader_2.54mm:PinHeader_1x06_P2.54mm_Vertical, symbol Connector:Conn_01x06_Male
- added J18, J19, J22: Conn_01x03_Male, Connector_JST:JST_PH_S3B-PH-K_1x03_P2.00mm_Horizontal, symbol Connector:Conn_01x03_Male
- added J24: Conn_02x02_Odd_Even, Connector_PinHeader_2.54mm:PinHeader_2x02_P2.54mm_Vertical, symbol Connector_Generic:Conn_02x02_Odd_Even
- added J5, J6, J7: Conn_01x02_Female, Sailboat:BAT-CONN, symbol Connector:Conn_01x02_Female
- D4, D5: footprint Diodes_THT:D_5W_P10.16mm_Horizontal -> Diode_THT:D_5W_P10.16mm_Horizontal; symbol D_Schottky -> Device:D_Schottky
Connections:
- net 5V-Rpi: now also J24.4 (Pin_4)
- net 5V-Sensors: now also J12.1 (Pin_1), J13.1 (Pin_1), J18.2 (Pin_2), J19.2 (Pin_2), J22.2 (Pin_2), J23.1 (Pin_1), J24.2 (Pin_2), J25.1 (Pin_1), J3.1 (Pin_1), J4.1 (Pin_1)
- net 5V-Servo: now also J1.2 (Pin_2), J14.2 (Pin_2), J15.2 (Pin_2), J2.2 (Pin_2)
- net A0: now also J18.3 (Pin_3)
- net A1: now also J19.3 (Pin_3)
- net A2: now also J22.3 (Pin_3)
- net BAT+: now also J10.1 (Pin_1), J11.1 (Pin_1)
- net BAT-: now also J10.2 (Pin_2), J11.2 (Pin_2), J6.1 (Pin_1), J7.1 (Pin_1)
- net CD_SD: now also J17.4 (Pin_4)
- net CS_SD: now also J17.5 (Pin_5)
- net D0: now also J20.2 (Pin_2)
- net D1: now also J21.2 (Pin_2)
- net GND: now also J1.3 (Pin_3), J12.2 (Pin_2), J13.2 (Pin_2), J14.3 (Pin_3), J15.3 (Pin_3), J18.1 (Pin_1), J19.1 (Pin_1), J2.3 (Pin_3), J20.1 (Pin_1), J21.1 (Pin_1), J22.1 (Pin_1), J23.2 (Pin_2), J24.1 (Pin_1), J24.3 (Pin_3), J25.2 (Pin_2), J3.2 (Pin_2), J4.2 (Pin_2)
- net MISO_SPI: now also J17.2 (Pin_2)
- net MOSI_SPI: now also J17.3 (Pin_3)
- net RC_1: now also J16.1 (Pin_1)
- net RC_2: now also J16.2 (Pin_2)
- net RC_3: now also J16.3 (Pin_3)
- net RC_4: now also J16.4 (Pin_4)
- net RC_5: now also J16.5 (Pin_5)
- net RC_6: now also J16.6 (Pin_6)
- net RX_1: now also J23.4 (Pin_4)
- net RX_2: now also J25.4 (Pin_4)
- net SCK_SPI: now also J17.1 (Pin_1)
- net SCL: now also J12.3 (Pin_3), J13.3 (Pin_3), J3.3 (Pin_3), J4.3 (Pin_3)
- net SDA: now also J12.4 (Pin_4), J13.4 (Pin_4), J3.4 (Pin_4), J4.4 (Pin_4)
- net Servo-1: now also J14.1 (Pin_1)
- net Servo-2: now also J15.1 (Pin_1)
- net Servo-Rudder: now also J2.1 (Pin_1)
- net Servo-Sail: now also J1.1 (Pin_1)
- net TX_1: now also J23.3 (Pin_3)
- net TX_2: now also J25.3 (Pin_3)
- net at D4.1 (K): now also J6.2 (Pin_2)
- net at D5.1 (K): now also J7.2 (Pin_2)
- new net: J5.1 (Pin_1), J8.1 (Pin_1), J9.1 (Pin_1)
- new net: J5.2 (Pin_2), J8.2 (Pin_2), J9.2 (Pin_2)
