File: Electronic Board/Sailboat Kicad/Board1-Arduino/Power.sch (KiCad schematic (older format))
At the start: 11 parts, among them U1 L7805, U2 L7805, U3 L7805

Commit message: Cleaned up, and added security, text and better usability, preparation for board v2
Parts:
- added D2, D3: D_Schottky, Diodes_THT:D_5W_P10.16mm_Horizontal, symbol D_Schottky
- added R4: 20k, Resistors_THT:R_Axial_DIN0204_L3.6mm_D1.6mm_P5.08mm_Horizontal, symbol R
- added R5: 12k, Resistors_THT:R_Axial_DIN0204_L3.6mm_D1.6mm_P5.08mm_Horizontal, symbol R
- L1, L2: footprint Inductors_THT:L_Axial_L5.3mm_D2.2mm_P7.62mm_Horizontal_Vishay_IM-1 -> Inductors_THT:L_Axial_L6.6mm_D2.7mm_P10.16mm_Horizontal_Vishay_IM-2
Connections:
- net 5V_Raspberry: now also D3.2 (A)
- net 5V_Servos: now also D2.2 (A)
- net BAT+: now also R4.1
- net GND: now also R5.2
- net at L1.1, U1.1 (IN): now also D3.1 (K)
- net at L2.1, U2.1 (IN): now also D2.1 (K)
- new net A3: R4.2, R5.1
Other:
- note added: "Battery tester :\n12V => 4.5V\n6V => 2.25V"
- moved on the sheet: C1, D1, L1, R1, U1
Changed lines of the file:
@@
 L GND #PWR03
 U 1 1 5A0C8A1D
-P 6900 1600
-F 0 "#PWR03" H 6900 1350 50  0001 C CNN
-F 1 "GND" H 6900 1450 50  0000 C CNN
-F 2 "" H 6900 1600 50  0001 C CNN
-F 3 "" H 6900 1600 50  0001 C CNN
-	1    6900 1600
+P 6900 1400
+F 0 "#PWR03" H 6900 1150 50  0001 C CNN
+F 1 "GND" H 6900 1250 50  0000 C CNN
+F 2 "" H 6900 1400 50  0001 C CNN
+F 3 "" H 6900 1400 50  0001 C CNN
+	1    6900 1400
 	0    -1   -1   0
 $EndComp
@@
 L R_Small R1
 U 1 1 5A0C8A34
-P 6400 1600
-F 0 "R1" H 6430 1620 50  0000 L CNN
-F 1 "330" H 6430 1560 50  0000 L CNN
-F 2 "Resistors_THT:R_Axial_DIN0204_L3.6mm_D1.6mm_P7.62mm_Horizontal" H 6400 1600 50  0001 C CNN
-F 3 "" H 6400 1600 50  0001 C CNN
-	1    6400 1600
+P 6400 1400
+F 0 "R1" H 6430 1420 50  0000 L CNN
+F 1 "330" H 6430 1360 50  0000 L CNN
+F 2 "Resistors_THT:R_Axial_DIN0204_L3.6mm_D1.6mm_P7.62mm_Horizontal" H 6400 1400 50  0001 C CNN
+F 3 "" H 6400 1400 50  0001 C CNN
+	1    6400 1400
 	0    1    1    0
 $EndComp
@@
 L LED_Small D1
 U 1 1 5A0C8A81
-P 6700 1600
-F 0 "D1" H 6650 1725 50  0000 L CNN
-F 1 "G" H 6525 1500 50  0000 L CNN
-F 2 "LEDs:LED_D3.0mm" V 6700 1600 50  0001 C CNN
-F 3 "" V 6700 1600 50  0001 C CNN
-	1    6700 1600
+P 6700 1400
+F 0 "D1" H 6650 1525 50  0000 L CNN
+F 1 "G" H 6525 1300 50  0000 L CNN
+F 2 "LEDs:LED_D3.0mm" V 6700 1400 50  0001 C CNN
+F 3 "" V 6700 1400 50  0001 C CNN
+	1    6700 1400
 	-1   0    0    1
 $EndComp
 Wire Wire Line
-	6900 1600 6800 1600
-Wire Wire Line
-	6600 1600 6500 1600
-Wire Wire Line
-	6300 1600 6200 1600
-Text GLabel 5800 2150 0    60   Input ~ 0
+	6900 1400 6800 1400
+Wire Wire Line
+	6600 1400 6500 1400
+Wire Wire Line
+	6300 1400 6200 1400
+Text GLabel 5800 2250 0    60   Input ~ 0
 BAT+
 $Comp
 L GND #PWR04
 U 1 1 5A0F1D5F
-P 6550 2550
-F 0 "#PWR04" H 6550 2300 50  0001 C CNN
-F 1 "GND" H 6550 2400 50  0000 C CNN
-F 2 "" H 6550 2550 50  0001 C CNN
-F 3 "" H 6550 2550 50  0001 C CNN
-	1    6550 2550
-	1    0    0    -1
-$EndComp
-Text HLabel 7300 2150 2    60   BiDi ~ 0
+P 6550 2650
+F 0 "#PWR04" H 6550 2400 50  0001 C CNN
+F 1 "GND" H 6550 2500 50  0000 C CNN
+F 2 "" H 6550 2650 50  0001 C CNN
+F 3 "" H 6550 2650 50  0001 C CNN
+	1    6550 2650
+	1    0    0    -1
+$EndComp
+Text HLabel 7300 2250 2    60   BiDi ~ 0
 5V_Raspberry
 $Comp
 L L7805 U1
 U 1 1 5A9587EC
-P 6550 2150
-F 0 "U1" H 6400 2275 50  0000 C CNN
-F 1 "L7805" H 6550 2275 50  0000 L CNN
-F 2 "TO_SOT_Packages_THT:TO-220-3_Vertical" H 6575 2000 50  0001 L CIN
-F 3 "" H 6550 2100 50  0001 C CNN
-	1    6550 2150
-	1    0    0    -1
-$EndComp
-Wire Wire Line
-	6550 2450 6550 2550
+P 6550 2250
+F 0 "U1" H 6400 2375 50  0000 C CNN
+F 1 "L7805" H 6550 2375 50  0000 L CNN
+F 2 "TO_SOT_Packages_THT:TO-220-3_Vertical" H 6575 2100 50  0001 L CIN
+F 3 "" H 6550 2200 50  0001 C CNN
+	1    6550 2250
+	1    0    0    -1
+$EndComp
+Wire Wire Line
+	6550 2550 6550 2650
 $Comp
 L L_Small L1
 U 1 1 5A95EA60
-P 6100 2150
-F 0 "L1" H 6130 2190 50  0000 L CNN
-F 1 "3.3uH" H 5850 2150 50  0000 L CNN
-F 2 "Inductors_THT:L_Axial_L5.3mm_D2.2mm_P7.62mm_Horizontal_Vishay_IM-1" H 6100 2150 50  0001 C CNN
-F 3 "" H 6100 2150 50  0001 C CNN
-	1    6100 2150
+P 6100 2250
+F 0 "L1" H 6130 2290 50  0000 L CNN
+F 1 "3.3uH" H 5850 2250 50  0000 L CNN
+F 2 "Inductors_THT:L_Axial_L6.6mm_D2.7mm_P10.16mm_Horizontal_Vishay_IM-2" H 6100 2250 50  0001 C CNN
+F 3 "" H 6100 2250 50  0001 C CNN
+	1    6100 2250
 	0    1    1    0
 $EndComp
 Wire Wire Line
-	6250 2150 6200 2150
-Wire Wire Line
-	5800 2150 6000 2150
-Wire Wire Line
-	5900 2350 5900 2450
-Wire Wire Line
-	5900 2450 6550 2450
-Connection ~ 5900 2150
+	6250 2250 6200 2250
+Wire Wire Line
+	5800 2250 6000 2250
+Wire Wire Line
+	5900 2450 5900 2550
+Wire Wire Line
+	5900 2550 6550 2550
+Connection ~ 5900 2250
 Text GLabel 5750 4950 0    60   Input ~ 0
 BAT+
@@
 F 0 "L2" H 6080 4990 50  0000 L CNN
 F 1 "3.3uH" H 5800 4950 50  0000 L CNN
-F 2 "Inductors_THT:L_Axial_L5.3mm_D2.2mm_P7.62mm_Horizontal_Vishay_IM-1" H 6050 4950 50  0001 C CNN
+F 2 "Inductors_THT:L_Axial_L6.6mm_D2.7mm_P10.16mm_Horizontal_Vishay_IM-2" H 6050 4950 50  0001 C CNN
 F 3 "" H 6050 4950 50  0001 C CNN
 	1    6050 4950
@@
 Connection ~ 5850 4950
 Wire Wire Line
-	7300 2150 6850 2150
+	7300 2250 6850 2250
 Wire Wire Line
 	7250 4950 6800 4950
@@
 Wire Wire Line
 	3300 2400 3100 2400
-Text HLabel 6200 1600 0    60   BiDi ~ 0
+Text HLabel 6200 1400 0    60   BiDi ~ 0
 5V_Raspberry
 $Comp
@@
 L C_Small C1
 U 1 1 5A958A75
-P 5900 2250
-F 0 "C1" H 5910 2320 50  0000 L CNN
-F 1 "4.7uF" H 5910 2170 50  0000 L CNN
-F 2 "Capacitors_THT:C_Rect_L7.0mm_W2.0mm_P5.00mm" H 5900 2250 50  0001 C CNN
-F 3 "" H 5900 2250 50  0001 C CNN
-	1    5900 2250
-	1    0    0    -1
-$EndComp
+P 5900 2350
+F 0 "C1" H 5910 2420 50  0000 L CNN
+F 1 "4.7uF" H 5910 2270 50  0000 L CNN
+F 2 "Capacitors_THT:C_Rect_L7.0mm_W2.0mm_P5.00mm" H 5900 2350 50  0001 C CNN
+F 3 "" H 5900 2350 50  0001 C CNN
+	1    5900 2350
+	1    0    0    -1
+$EndComp
+Wire Wire Line
+	7050 2250 7050 1950
+Wire Wire Line
+	7050 1950 6700 1950
+Connection ~ 7050 2250
+Wire Wire Line
+	6400 1950 6250 1950
+Wire Wire Line
+	6250 1950 6250 2250
+Wire Wire Line
+	7000 4950 7000 4600
+Wire Wire Line
+	7000 4600 6650 4600
+Connection ~ 7000 4950
+Wire Wire Line
+	6350 4600 6200 4600
+Wire Wire Line
+	6200 4600 6200 4950
+$Comp
+L D_Schottky D3
+U 1 1 5B0DEFFA
+P 6550 1950
+F 0 "D3" H 6550 2050 50  0000 C CNN
+F 1 "D_Schottky" H 6550 1850 50  0000 C CNN
+F 2 "Diodes_THT:D_5W_P10.16mm_Horizontal" H 6550 1950 50  0001 C CNN
+F 3 "" H 6550 1950 50  0001 C CNN
+	1    6550 1950
+	1    0    0    -1
+$EndComp
+$Comp
+L D_Schottky D2
+U 1 1 5B0DF065
+P 6500 4600
+F 0 "D2" H 6500 4700 50  0000 C CNN
+F 1 "D_Schottky" H 6500 4500 50  0000 C CNN
+F 2 "Diodes_THT:D_5W_P10.16mm_Horizontal" H 6500 4600 50  0001 C CNN
+F 3 "" H 6500 4600 50  0001 C CNN
+	1    6500 4600
+	1    0    0    -1
+$EndComp
+Text GLabel 3100 3500 0    60   Input ~ 0
+BAT+
+$Comp
+L R R4
+U 1 1 5B0ED277
+P 3400 3650
+F 0 "R4" V 3480 3650 50  0000 C CNN
+F 1 "20k" V 3400 3650 50  0000 C CNN
+F 2 "Resistors_THT:R_Axial_DIN0204_L3.6mm_D1.6mm_P5.08mm_Horizontal" V 3330 3650 50  0001 C CNN
+F 3 "" H 3400 3650 50  0001 C CNN
+	1    3400 3650
+	1    0    0    -1
+$EndComp
+$Comp
+L R R5
+U 1 1 5B0ED326
+P 3400 4200
+F 0 "R5" V 3480 4200 50  0000 C CNN
+F 1 "12k" V 3400 4200 50  0000 C CNN
+F 2 "Resistors_THT:R_Axial_DIN0204_L3.6mm_D1.6mm_P5.08mm_Horizontal" V 3330 4200 50  0001 C CNN
+F 3 "" H 3400 4200 50  0001 C CNN
+	1    3400 4200
+	1    0    0    -1
+$EndComp
+$Comp
+L GND #PWR07
+U 1 1 5B0ED454
+P 3100 4350
+F 0 "#PWR07" H 3100 4100 50  0001 C CNN
+F 1 "GND" H 3100 4200 50  0000 C CNN
+F 2 "" H 3100 4350 50  0001 C CNN
+F 3 "" H 3100 4350 50  0001 C CNN
+	1    3100 4350
+	0    1    1    0
+$EndComp
+Wire Wire Line
+	3100 3500 3400 3500
+Wire Wire Line
+	3400 3800 3400 4050
+Wire Wire Line
+	3400 4350 3100 4350
+Text HLabel 3550 3900 2    60   BiDi ~ 0
+A3
+Wire Wire Line
+	3550 3900 3400 3900
+Connection ~ 3400 3900
+Text Notes 2800 3350 0    60   ~ 0
+Battery tester :\n12V => 4.5V\n6V => 2.25V
 $EndSCHEMATC

Commit message: added decoupler capacitor for voltage measurements and added connectors to arduino
Parts:
- added C5: 1uF, Capacitors_THT:C_Rect_L7.0mm_W2.0mm_P5.00mm, symbol C_Small
Connections:
- net A3: now also C5.1
- net GND: now also C5.2
Changed lines of the file:
@@
 	3400 3800 3400 4050
 Wire Wire Line
-	3400 4350 3100 4350
-Text HLabel 3550 3900 2    60   BiDi ~ 0
+	3100 4350 3650 4350
+Text HLabel 3700 3900 2    60   BiDi ~ 0
 A3
 Wire Wire Line
-	3550 3900 3400 3900
+	3400 3900 3700 3900
 Connection ~ 3400 3900
 Text Notes 2800 3350 0    60   ~ 0
 Battery tester :\n12V => 4.5V\n6V => 2.25V
+$Comp
+L C_Small C5
+U 1 1 5B9AD1C3
+P 3650 4200
+F 0 "C5" H 3660 4270 50  0000 L CNN
+F 1 "1uF" H 3660 4120 50  0000 L CNN
+F 2 "Capacitors_THT:C_Rect_L7.0mm_W2.0mm_P5.00mm" H 3650 4200 50  0001 C CNN
+F 3 "" H 3650 4200 50  0001 C CNN
+	1    3650 4200
+	1    0    0    -1
+$EndComp
+Wire Wire Line
+	3650 3900 3650 4100
+Connection ~ 3650 3900
+Wire Wire Line
+	3650 4350 3650 4300
+Connection ~ 3400 4350
 $EndSCHEMATC

Commit message: Updated version of Kicad, rendered images and BOM
Parts:
- removed U1, U2, U3: L7805, TO_SOT_Packages_THT:TO-220-3_Vertical, symbol L7805
- added U1, U2, U3: L7805, Package_TO_SOT_THT:TO-220-3_Vertical, symbol Regulator_Linear:L7805
- C1, C2, C5: footprint Capacitors_THT:C_Rect_L7.0mm_W2.0mm_P5.00mm -> Capacitor_THT:C_Rect_L7.0mm_W2.0mm_P5.00mm; symbol C_Small -> Device:C_Small
- C3, C4: footprint Capacitors_THT:C_Rect_L7.0mm_W3.5mm_P5.00mm -> Capacitor_THT:C_Rect_L7.0mm_W2.0mm_P5.00mm; symbol C_Small -> Device:C_Small
- D1: symbol LED_Small -> Device:LED_Small
- D2, D3: footprint Diodes_THT:D_5W_P10.16mm_Horizontal -> Diode_THT:D_5W_P10.16mm_Horizontal; symbol D_Schottky -> Device:D_Schottky
- L1, L2: footprint Inductors_THT:L_Axial_L6.6mm_D2.7mm_P10.16mm_Horizontal_Vishay_IM-2 -> Inductor_THT:L_Axial_L5.3mm_D2.2mm_P7.62mm_Horizontal_Vishay_IM-1; symbol L_Small -> Device:L_Small
- R1: footprint Resistors_THT:R_Axial_DIN0204_L3.6mm_D1.6mm_P7.62mm_Horizontal -> Resistor_THT:R_Axial_DIN0204_L3.6mm_D1.6mm_P7.62mm_Horizontal; symbol R_Small -> Device:R_Small
- R4, R5: footprint Resistors_THT:R_Axial_DIN0204_L3.6mm_D1.6mm_P5.08mm_Horizontal -> Resistor_THT:R_Axial_DIN0204_L3.6mm_D1.6mm_P7.62mm_Horizontal; symbol R -> Device:R
Connections:
- net 5V_Raspberry: now also U2.3 (OUT)
- net 5V_Sensors: now also U3.3 (OUT)
- net 5V_Servos: now also U1.3 (OUT)
- net BAT+: now also U3.1 (IN)
- net GND: now also U1.2 (GND), U2.2 (GND), U3.2 (GND)
- net at D3.1 (K), L1.1: now also U2.1 (IN)
- net at D2.1 (K), L2.1: now also U1.1 (IN)
Changed lines of the file:
@@
-EESchema Schematic File Version 2
-LIBS:power
-LIBS:device
-LIBS:switches
-LIBS:relays
-LIBS:motors
-LIBS:transistors
-LIBS:conn
-LIBS:linear
-LIBS:regul
-LIBS:74xx
-LIBS:cmos4000
-LIBS:adc-dac
-LIBS:memory
-LIBS:xilinx
-LIBS:microcontrollers
-LIBS:dsp
-LIBS:microchip
-LIBS:analog_switches
-LIBS:motorola
-LIBS:texas
-LIBS:intel
-LIBS:audio
-LIBS:interface
-LIBS:digital-audio
-LIBS:philips
-LIBS:display
-LIBS:cypress
-LIBS:siliconi
-LIBS:opto
-LIBS:atmel
-LIBS:contrib
-LIBS:valves
+EESchema Schematic File Version 4
 LIBS:Arduino Interface-cache
-EELAYER 25 0
+EELAYER 26 0
 EELAYER END
 $Descr A4 11693 8268
@@
 	3100 2300 3300 2300
 $Comp
-L GND #PWR02
+L power:GND #PWR02
 U 1 1 5A0C377E
 P 3300 2400
@@
 BAT-
 $Comp
-L GND #PWR03
+L power:GND #PWR03
 U 1 1 5A0C8A1D
 P 6900 1400
@@
 $EndComp
 $Comp
-L R_Small R1
+L Device:R_Small R1
 U 1 1 5A0C8A34
 P 6400 1400
 F 0 "R1" H 6430 1420 50  0000 L CNN
 F 1 "330" H 6430 1360 50  0000 L CNN
-F 2 "Resistors_THT:R_Axial_DIN0204_L3.6mm_D1.6mm_P7.62mm_Horizontal" H 6400 1400 50  0001 C CNN
+F 2 "Resistor_THT:R_Axial_DIN0204_L3.6mm_D1.6mm_P7.62mm_Horizontal" H 6400 1400 50  0001 C CNN
 F 3 "" H 6400 1400 50  0001 C CNN
 	1    6400 1400
@@
 $EndComp
 $Comp
-L LED_Small D1
+L Device:LED_Small D1
 U 1 1 5A0C8A81
 P 6700 1400
@@
 BAT+
 $Comp
-L GND #PWR04
+L power:GND #PWR04
 U 1 1 5A0F1D5F
 P 6550 2650
@@
 Text HLabel 7300 2250 2    60   BiDi ~ 0
 5V_Raspberry
-$Comp
-L L7805 U1
-U 1 1 5A9587EC
-P 6550 2250
-F 0 "U1" H 6400 2375 50  0000 C CNN
-F 1 "L7805" H 6550 2375 50  0000 L CNN
-F 2 "TO_SOT_Packages_THT:TO-220-3_Vertical" H 6575 2100 50  0001 L CIN
-F 3 "" H 6550 2200 50  0001 C CNN
-	1    6550 2250
-	1    0    0    -1
-$EndComp
 Wire Wire Line
 	6550 2550 6550 2650
 $Comp
-L L_Small L1
+L Device:L_Small L1
 U 1 1 5A95EA60
 P 6100 2250
 F 0 "L1" H 6130 2290 50  0000 L CNN
 F 1 "3.3uH" H 5850 2250 50  0000 L CNN
-F 2 "Inductors_THT:L_Axial_L6.6mm_D2.7mm_P10.16mm_Horizontal_Vishay_IM-2" H 6100 2250 50  0001 C CNN
+F 2 "Inductor_THT:L_Axial_L5.3mm_D2.2mm_P7.62mm_Horizontal_Vishay_IM-1" H 6100 2250 50  0001 C CNN
 F 3 "" H 6100 2250 50  0001 C CNN
 	1    6100 2250
@@
 	6250 2250 6200 2250
 Wire Wire Line
-	5800 2250 6000 2250
+	5800 2250 5900 2250
 Wire Wire Line
 	5900 2450 5900 2550
@@
 BAT+
 $Comp
-L GND #PWR05
+L power:GND #PWR05
 U 1 1 5A960D95
 P 6500 5350
@@
 Text HLabel 7250 4950 2    60   BiDi ~ 0
 5V_Servos
-$Comp
-L L7805 U2
-U 1 1 5A960D9C
-P 6500 4950
-F 0 "U2" H 6350 5075 50  0000 C CNN
-F 1 "L7805" H 6500 5075 50  0000 L CNN
-F 2 "TO_SOT_Packages_THT:TO-220-3_Vertical" H 6525 4800 50  0001 L CIN
-F 3 "" H 6500 4900 50  0001 C CNN
-	1    6500 4950
-	1    0    0    -1
-$EndComp
 Wire Wire Line
 	6500 5250 6500 5350
 $Comp
-L L_Small L2
+L Device:L_Small L2
 U 1 1 5A960DAC
 P 6050 4950
 F 0 "L2" H 6080 4990 50  0000 L CNN
 F 1 "3.3uH" H 5800 4950 50  0000 L CNN
-F 2 "Inductors_THT:L_Axial_L6.6mm_D2.7mm_P10.16mm_Horizontal_Vishay_IM-2" H 6050 4950 50  0001 C CNN
+F 2 "Inductor_THT:L_Axial_L5.3mm_D2.2mm_P7.62mm_Horizontal_Vishay_IM-1" H 6050 4950 50  0001 C CNN
 F 3 "" H 6050 4950 50  0001 C CNN
 	1    6050 4950
@@
 	6200 4950 6150 4950
 Wire Wire Line
-	5750 4950 5950 4950
+	5750 4950 5850 4950
 Wire Wire Line
 	5850 5150 5850 5250
@@
 Connection ~ 5850 4950
 Wire Wire Line
-	7300 2250 6850 2250
-Wire Wire Line
-	7250 4950 6800 4950
-$Comp
-L L7805 U3
-U 1 1 5A97895C
-P 6600 3500
-F 0 "U3" H 6450 3625 50  0000 C CNN
-F 1 "L7805" H 6600 3625 50  0000 L CNN
-F 2 "TO_SOT_Packages_THT:TO-220-3_Vertical" H 6625 3350 50  0001 L CIN
-F 3 "" H 6600 3450 50  0001 C CNN
-	1    6600 3500
-	1    0    0    -1
-$EndComp
-$Comp
-L GND #PWR06
+	7300 2250 7050 2250
+Wire Wire Line
+	7250 4950 7000 4950
+$Comp
+L power:GND #PWR06
 U 1 1 5A9789B4
 P 6600 3900
@@
 $EndComp
 $Comp
-L C_Small C3
+L Device:C_Small C3
 U 1 1 5A9789DA
 P 6150 3600
 F 0 "C3" H 6160 3670 50  0000 L CNN
 F 1 "0.33uF" H 6160 3520 50  0000 L CNN
-F 2 "Capacitors_THT:C_Rect_L7.0mm_W3.5mm_P5.00mm" H 6150 3600 50  0001 C CNN
+F 2 "Capacitor_THT:C_Rect_L7.0mm_W2.0mm_P5.00mm" H 6150 3600 50  0001 C CNN
 F 3 "" H 6150 3600 50  0001 C CNN
 	1    6150 3600
@@
 $EndComp
 $Comp
-L C_Small C4
+L Device:C_Small C4
 U 1 1 5A978A20
 P 7050 3600
 F 0 "C4" H 7060 3670 50  0000 L CNN
 F 1 "0.1uF" H 7060 3520 50  0000 L CNN
-F 2 "Capacitors_THT:C_Rect_L7.0mm_W3.5mm_P5.00mm" H 7050 3600 50  0001 C CNN
+F 2 "Capacitor_THT:C_Rect_L7.0mm_W2.0mm_P5.00mm" H 7050 3600 50  0001 C CNN
 F 3 "" H 7050 3600 50  0001 C CNN
 	1    7050 3600
@@
 $EndComp
 Wire Wire Line
-	5900 3500 6300 3500
+	5900 3500 6150 3500
 Connection ~ 6150 3500
 Wire Wire Line
 	6150 3700 6150 3800
 Wire Wire Line
-	6150 3800 7050 3800
+	6150 3800 6600 3800
 Wire Wire Line
 	7050 3800 7050 3700
 Connection ~ 6600 3800
 Wire Wire Line
-	6900 3500 7300 3500
+	6900 3500 7050 3500
 Wire Wire Line
 	6600 3900 6600 3800
@@
 5V_Raspberry
 $Comp
-L C_Small C2
+L Device:C_Small C2
 U 1 1 5A960DA2
 P 5850 5050
 F 0 "C2" H 5860 5120 50  0000 L CNN
 F 1 "4.7uF" H 5860 4970 50  0000 L CNN
-F 2 "Capacitors_THT:C_Rect_L7.0mm_W2.0mm_P5.00mm" H 5850 5050 50  0001 C CNN
+F 2 "Capacitor_THT:C_Rect_L7.0mm_W2.0mm_P5.00mm" H 5850 5050 50  0001 C CNN
 F 3 "" H 5850 5050 50  0001 C CNN
 	1    5850 5050
@@
 $EndComp
 $Comp
-L C_Small C1
+L Device:C_Small C1
 U 1 1 5A958A75
 P 5900 2350
 F 0 "C1" H 5910 2420 50  0000 L CNN
 F 1 "4.7uF" H 5910 2270 50  0000 L CNN
-F 2 "Capacitors_THT:C_Rect_L7.0mm_W2.0mm_P5.00mm" H 5900 2350 50  0001 C CNN
+F 2 "Capacitor_THT:C_Rect_L7.0mm_W2.0mm_P5.00mm" H 5900 2350 50  0001 C CNN
 F 3 "" H 5900 2350 50  0001 C CNN
 	1    5900 2350
@@
 	6200 4600 6200 4950
 $Comp
-L D_Schottky D3
+L Device:D_Schottky D3
 U 1 1 5B0DEFFA
 P 6550 1950
 F 0 "D3" H 6550 2050 50  0000 C CNN
 F 1 "D_Schottky" H 6550 1850 50  0000 C CNN
-F 2 "Diodes_THT:D_5W_P10.16mm_Horizontal" H 6550 1950 50  0001 C CNN
+F 2 "Diode_THT:D_5W_P10.16mm_Horizontal" H 6550 1950 50  0001 C CNN
 F 3 "" H 6550 1950 50  0001 C CNN
 	1    6550 1950
@@
 $EndComp
 $Comp
-L D_Schottky D2
+L Device:D_Schottky D2
 U 1 1 5B0DF065
 P 6500 4600
 F 0 "D2" H 6500 4700 50  0000 C CNN
 F 1 "D_Schottky" H 6500 4500 50  0000 C CNN
-F 2 "Diodes_THT:D_5W_P10.16mm_Horizontal" H 6500 4600 50  0001 C CNN
+F 2 "Diode_THT:D_5W_P10.16mm_Horizontal" H 6500 4600 50  0001 C CNN
 F 3 "" H 6500 4600 50  0001 C CNN
 	1    6500 4600
@@
 BAT+
 $Comp
-L R R4
+L Device:R R4
 U 1 1 5B0ED277
 P 3400 3650
 F 0 "R4" V 3480 3650 50  0000 C CNN
 F 1 "20k" V 3400 3650 50  0000 C CNN
-F 2 "Resistors_THT:R_Axial_DIN0204_L3.6mm_D1.6mm_P5.08mm_Horizontal" V 3330 3650 50  0001 C CNN
+F 2 "Resistor_THT:R_Axial_DIN0204_L3.6mm_D1.6mm_P7.62mm_Horizontal" V 3330 3650 50  0001 C CNN
 F 3 "" H 3400 3650 50  0001 C CNN
 	1    3400 3650
@@
 $EndComp
 $Comp
-L R R5
+L Device:R R5
 U 1 1 5B0ED326
 P 3400 4200
 F 0 "R5" V 3480 4200 50  0000 C CNN
 F 1 "12k" V 3400 4200 50  0000 C CNN
-F 2 "Resistors_THT:R_Axial_DIN0204_L3.6mm_D1.6mm_P5.08mm_Horizontal" V 3330 4200 50  0001 C CNN
+F 2 "Resistor_THT:R_Axial_DIN0204_L3.6mm_D1.6mm_P7.62mm_Horizontal" V 3330 4200 50  0001 C CNN
 F 3 "" H 3400 4200 50  0001 C CNN
 	1    3400 4200
@@
 $EndComp
 $Comp
-L GND #PWR07
+L power:GND #PWR07
 U 1 1 5B0ED454
 P 3100 4350
@@
 	3100 3500 3400 3500
 Wire Wire Line
-	3400 3800 3400 4050
-Wire Wire Line
-	3100 4350 3650 4350
+	3400 3800 3400 3900
+Wire Wire Line
+	3100 4350 3400 4350
 Text HLabel 3700 3900 2    60   BiDi ~ 0
 A3
 Wire Wire Line
-	3400 3900 3700 3900
+	3400 3900 3650 3900
 Connection ~ 3400 3900
 Text Notes 2800 3350 0    60   ~ 0
 Battery tester :\n12V => 4.5V\n6V => 2.25V
 $Comp
-L C_Small C5
+L Device:C_Small C5
 U 1 1 5B9AD1C3
 P 3650 4200
 F 0 "C5" H 3660 4270 50  0000 L CNN
 F 1 "1uF" H 3660 4120 50  0000 L CNN
-F 2 "Capacitors_THT:C_Rect_L7.0mm_W2.0mm_P5.00mm" H 3650 4200 50  0001 C CNN
+F 2 "Capacitor_THT:C_Rect_L7.0mm_W2.0mm_P5.00mm" H 3650 4200 50  0001 C CNN
 F 3 "" H 3650 4200 50  0001 C CNN
 	1    3650 4200
@@
 	3650 4350 3650 4300
 Connection ~ 3400 4350
+Wire Wire Line
+	5900 2250 6000 2250
+Wire Wire Line
+	5850 4950 5950 4950
+Wire Wire Line
+	6150 3500 6300 3500
+Wire Wire Line
+	6600 3800 7050 3800
+Wire Wire Line
+	7050 3500 7300 3500
+Wire Wire Line
+	7050 2250 6850 2250
+Wire Wire Line
+	7000 4950 6800 4950
+Wire Wire Line
+	3400 3900 3400 4050
+Wire Wire Line
+	3650 3900 3700 3900
+Wire Wire Line
+	3400 4350 3650 4350
+$Comp
+L Regulator_Linear:L7805 U2
+U 1 1 5D0032D4
+P 6550 2250
+F 0 "U2" H 6550 2492 50  0000 C CNN
+F 1 "L7805" H 6550 2401 50  0000 C CNN
+F 2 "Package_TO_SOT_THT:TO-220-3_Vertical" H 6575 2100 50  0001 L CIN
+F 3 "http://www.st.com/content/ccc/resource/technical/document/datasheet/41/4f/b3/b0/12/d4/47/88/CD00000444.pdf/files/CD00000444.pdf/jcr:content/translations/en.CD00000444.pdf" H 6550 2200 50  0001 C CNN
+	1    6550 2250
+	1    0    0    -1
+$EndComp
+Connection ~ 6250 2250
+Connection ~ 6550 2550
+$Comp
+L Regulator_Linear:L7805 U3
+U 1 1 5D0033D0
+P 6600 3500
+F 0 "U3" H 6600 3742 50  0000 C CNN
+F 1 "L7805" H 6600 3651 50  0000 C CNN
+F 2 "Package_TO_SOT_THT:TO-220-3_Vertical" H 6625 3350 50  0001 L CIN
+F 3 "http://www.st.com/content/ccc/resource/technical/document/datasheet/41/4f/b3/b0/12/d4/47/88/CD00000444.pdf/files/CD00000444.pdf/jcr:content/translations/en.CD00000444.pdf" H 6600 3450 50  0001 C CNN
+	1    6600 3500
+	1    0    0    -1
+$EndComp
+$Comp
+L Regulator_Linear:L7805 U1
+U 1 1 5D00342A
+P 6500 4950
+F 0 "U1" H 6500 5192 50  0000 C CNN
+F 1 "L7805" H 6500 5101 50  0000 C CNN
+F 2 "Package_TO_SOT_THT:TO-220-3_Vertical" H 6525 4800 50  0001 L CIN
+F 3 "http://www.st.com/content/ccc/resource/technical/document/datasheet/41/4f/b3/b0/12/d4/47/88/CD00000444.pdf/files/CD00000444.pdf/jcr:content/translations/en.CD00000444.pdf" H 6500 4900 50  0001 C CNN
+	1    6500 4950
+	1    0    0    -1
+$EndComp
+Connection ~ 6200 4950
+Connection ~ 6500 5250
 $EndSCHEMATC
