File: Electronic Board/Sailboat Kicad/Board2-RPI/RPi Interface.kicad_pcb (KiCad board)
At the start: 2 copper layers, 70.5 x 100.3 mm, 18 parts, among them J1 Conn_01x06, J2 Conn_01x06, J23 Conn_02x20_Odd_Even, J25 Conn_01x03_Female, J26 Conn_01x03_Female, J27 Conn_01x03_Female, J28 Conn_01x03_Female, J29 Conn_01x03_Female, J3 Conn_02x02_Odd_Even, J30 Conn_01x03_Female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

Commit message: Finished board-v0.1
Parts:
- removed the REF** at (184.2, 59.7)
- removed the REF** at (177.2, 55.9)
- removed the REF** at (128.9, 55.9)
- removed the REF** at (135.3, 59.7)
- removed the REF** at (184.2, 118.1)
- removed the REF** at (135.3, 118.1)
- removed the REF** at (177.2, 137.2)
- added J4: Conn_01x03_Female, Socket_Strips:Socket_Strip_Straight_1x03_Pitch2.54mm, F.Cu at (139.1, 123.2)
- added REF**: MountingHole_3.2mm_M3, Mounting_Holes:MountingHole_3.2mm_M3, F.Cu at (184.2, 59.7)
- added REF**: MountingHole_3.2mm_M3, Mounting_Holes:MountingHole_3.2mm_M3, F.Cu at (128.9, 55.9)
- added REF**: MountingHole_3.2mm_M3, Mounting_Holes:MountingHole_3.2mm_M3, F.Cu at (135.3, 59.7)
- added REF**: MountingHole_3.2mm_M3, Mounting_Holes:MountingHole_3.2mm_M3, F.Cu at (135.3, 118.1)
- added REF**: MountingHole_3.2mm_M3, Mounting_Holes:MountingHole_3.2mm_M3, F.Cu at (184.2, 118.1)
- added REF**: MountingHole_3.2mm_M3, Mounting_Holes:MountingHole_3.2mm_M3, F.Cu at (177.2, 137.2)
Routing:
- net 5V-Sensors: track 100.5 -> 238.1 mm
- net GND: track 0.00 -> 20.5 mm
- net /Connectors/5V-RPi: track 143.8 -> 140.5 mm
Other:
- board size 70.5 x 100.3 mm -> 69.9 x 99.1 mm
