File: Electronic Board/Sailboat Kicad/Board2-RPI/RPi Interface.kicad_pcb (KiCad board)
At the start: 2 copper layers, 69.9 x 99.1 mm, 21 parts, among them J1 Conn_01x06, J2 Conn_01x06, J23 Conn_02x20_Odd_Even, J25 Conn_01x03_Female, J26 Conn_01x03_Female, J27 Conn_01x03_Female, J28 Conn_01x03_Female, J29 Conn_01x03_Female, J3 Conn_02x02_Odd_Even, J30 Conn_01x03_Female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

Commit message: Minor changes and recompiled gerber, pdf and 3D
Other:
- outline, holes or cut-outs redrawn
Changed lines of the file:
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@@
     (area 113.902618 36.094999 193.707143 157.020239)
     (thickness 1.6)
-    (drawings 36)
+    (drawings 35)
     (tracks 209)
     (zones 0)
@@
     (pcbplotparams
       (layerselection 0x010f0_80000001)
-      (usegerberextensions true)
+      (usegerberextensions false)
       (excludeedgelayer true)
       (linewidth 0.100000)
@@
       (padsonsilk false)
       (subtractmaskfromsilk false)
-      (outputformat 1)
+      (outputformat 4)
       (mirror false)
       (drillshape 0)
       (scaleselection 1)
-      (outputdirectory Gerber/))
+      (outputdirectory PDF/))
   )
   (net 0 "")
@@
     (add_net SCK_SPI)
   )
+  (module Mounting_Holes:MountingHole_3.2mm_M3 (layer F.Cu)
+    (at 184.15 59.69)
+    (descr "Mounting Hole 3.2mm, no annular, M3")
+    (tags "mounting hole 3.2mm no annular m3")
+    (attr virtual)
+    (fp_text reference REF** (at 0 -4.2) (layer F.SilkS)
+      (effects (font (size 1 1) (thickness 0.15)))
+    )
+    (fp_text value MountingHole_3.2mm_M3 (at 0 4.2) (layer F.Fab)
+      (effects (font (size 1 1) (thickness 0.15)))
+    )
+    (fp_text user %R (at 0.3 0) (layer F.Fab)
+      (effects (font (size 1 1) (thickness 0.15)))
+    )
+    (fp_circle (center 0 0) (end 3.2 0) (layer Cmts.User) (width 0.15))
+    (fp_circle (center 0 0) (end 3.45 0) (layer F.CrtYd) (width 0.05))
+    (pad 1 np_thru_hole circle (at 0 0) (size 3.2 3.2) (drill 3.2) (layers *.Cu *.Mask))
+  )
   (module Socket_Strips:Socket_Strip_Straight_1x03_Pitch2.54mm (layer B.Cu)
     (at 139.065 144.145 90)
@@
       (rotate (xyz 0 0 270))
     )
-  )
-  (module Mounting_Holes:MountingHole_3.2mm_M3 (layer F.Cu)
-    (at 184.15 59.69)
-    (descr "Mounting Hole 3.2mm, no annular, M3")
-    (tags "mounting hole 3.2mm no annular m3")
-    (attr virtual)
-    (fp_text reference REF** (at 0 -4.2) (layer F.SilkS)
-      (effects (font (size 1 1) (thickness 0.15)))
-    )
-    (fp_text value MountingHole_3.2mm_M3 (at 0 4.2) (layer F.Fab)
-      (effects (font (size 1 1) (thickness 0.15)))
-    )
-    (fp_text user %R (at 0.3 0) (layer F.Fab)
-      (effects (font (size 1 1) (thickness 0.15)))
-    )
-    (fp_circle (center 0 0) (end 3.2 0) (layer Cmts.User) (width 0.15))
-    (fp_circle (center 0 0) (end 3.45 0) (layer F.CrtYd) (width 0.05))
-    (pad 1 np_thru_hole circle (at 0 0) (size 3.2 3.2) (drill 3.2) (layers *.Cu *.Mask))
   )
   (module Socket_Strips:Socket_Strip_Straight_1x08_Pitch2.54mm (layer B.Cu)
@@
     (pad 1 np_thru_hole circle (at 0 0) (size 3.2 3.2) (drill 3.2) (layers *.Cu *.Mask))
   )
-  (gr_line (start 187.96 53.34) (end 187.96 57.15) (angle 90) (layer Edge.Cuts) (width 0.1))
+  (gr_line (start 173.355 61.595) (end 173.355 77.47) (angle 90) (layer Edge.Cuts) (width 0.1))
+  (gr_line (start 187.96 61.595) (end 173.355 61.595) (angle 90) (layer Edge.Cuts) (width 0.1))
+  (gr_line (start 187.96 53.34) (end 187.96 61.595) (angle 90) (layer Edge.Cuts) (width 0.1))
   (gr_line (start 160.02 53.34) (end 187.96 53.34) (angle 90) (layer Edge.Cuts) (width 0.1))
   (gr_line (start 118.11 152.4) (end 187.96 152.4) (angle 90) (layer Edge.Cuts) (width 0.1))
@@
   (gr_line (start 118.11 53.34) (end 118.11 152.4) (angle 90) (layer Edge.Cuts) (width 0.1))
   (gr_line (start 173.355 77.47) (end 158.115 77.47) (angle 90) (layer Edge.Cuts) (width 0.1))
-  (gr_line (start 173.355 62.23) (end 173.355 77.47) (angle 90) (layer Edge.Cuts) (width 0.1))
-  (gr_line (start 187.96 62.23) (end 173.355 62.23) (angle 90) (layer Edge.Cuts) (width 0.1))
-  (gr_line (start 187.96 57.15) (end 187.96 62.23) (angle 90) (layer Edge.Cuts) (width 0.1))
   (gr_line (start 158.115 114.935) (end 158.115 77.47) (angle 90) (layer Edge.Cuts) (width 0.1))
   (gr_line (start 187.96 114.935) (end 158.115 114.935) (angle 90) (layer Edge.Cuts) (width 0.1))

Commit message: New board bug fix
Parts:
- removed the REF** at (184.2, 59.7)
- removed the REF** at (177.2, 54.6)
Other:
- outline, holes or cut-outs redrawn
Changed lines of the file:
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@@
     (area 113.902618 36.094999 193.707143 157.020239)
     (thickness 1.6)
-    (drawings 35)
+    (drawings 34)
     (tracks 209)
     (zones 0)
-    (modules 21)
+    (modules 19)
     (nets 56)
   )
@@
     (pcbplotparams
       (layerselection 0x010f0_80000001)
-      (usegerberextensions false)
+      (usegerberextensions true)
       (excludeedgelayer true)
       (linewidth 0.100000)
@@
       (padsonsilk false)
       (subtractmaskfromsilk false)
-      (outputformat 4)
+      (outputformat 1)
       (mirror false)
       (drillshape 0)
       (scaleselection 1)
-      (outputdirectory PDF/))
+      (outputdirectory Gerber/))
   )
   (net 0 "")
@@
     (add_net SCK_SPI)
   )
-  (module Mounting_Holes:MountingHole_3.2mm_M3 (layer F.Cu)
-    (at 184.15 59.69)
-    (descr "Mounting Hole 3.2mm, no annular, M3")
-    (tags "mounting hole 3.2mm no annular m3")
-    (attr virtual)
-    (fp_text reference REF** (at 0 -4.2) (layer F.SilkS)
-      (effects (font (size 1 1) (thickness 0.15)))
-    )
-    (fp_text value MountingHole_3.2mm_M3 (at 0 4.2) (layer F.Fab)
-      (effects (font (size 1 1) (thickness 0.15)))
-    )
-    (fp_text user %R (at 0.3 0) (layer F.Fab)
-      (effects (font (size 1 1) (thickness 0.15)))
-    )
-    (fp_circle (center 0 0) (end 3.2 0) (layer Cmts.User) (width 0.15))
-    (fp_circle (center 0 0) (end 3.45 0) (layer F.CrtYd) (width 0.05))
-    (pad 1 np_thru_hole circle (at 0 0) (size 3.2 3.2) (drill 3.2) (layers *.Cu *.Mask))
-  )
   (module Socket_Strips:Socket_Strip_Straight_1x03_Pitch2.54mm (layer B.Cu)
     (at 139.065 144.145 90)
@@
     (pad 1 np_thru_hole circle (at 0 0) (size 3.2 3.2) (drill 3.2) (layers *.Cu *.Mask))
   )
-  (module Mounting_Holes:MountingHole_3.2mm_M3 (layer F.Cu)
-    (at 177.165 54.61)
-    (descr "Mounting Hole 3.2mm, no annular, M3")
-    (tags "mounting hole 3.2mm no annular m3")
-    (attr virtual)
-    (fp_text reference REF** (at 0 -4.2) (layer F.SilkS)
-      (effects (font (size 1 1) (thickness 0.15)))
-    )
-    (fp_text value MountingHole_3.2mm_M3 (at 0 4.2) (layer F.Fab)
-      (effects (font (size 1 1) (thickness 0.15)))
-    )
-    (fp_text user %R (at 0.3 0) (layer F.Fab)
-      (effects (font (size 1 1) (thickness 0.15)))
-    )
-    (fp_circle (center 0 0) (end 3.2 0) (layer Cmts.User) (width 0.15))
-    (fp_circle (center 0 0) (end 3.45 0) (layer F.CrtYd) (width 0.05))
-    (pad 1 np_thru_hole circle (at 0 0) (size 3.2 3.2) (drill 3.2) (layers *.Cu *.Mask))
-  )
-  (gr_line (start 173.355 61.595) (end 173.355 77.47) (angle 90) (layer Edge.Cuts) (width 0.1))
-  (gr_line (start 187.96 61.595) (end 173.355 61.595) (angle 90) (layer Edge.Cuts) (width 0.1))
-  (gr_line (start 187.96 53.34) (end 187.96 61.595) (angle 90) (layer Edge.Cuts) (width 0.1))
-  (gr_line (start 160.02 53.34) (end 187.96 53.34) (angle 90) (layer Edge.Cuts) (width 0.1))
+  (gr_line (start 170.815 77.47) (end 158.115 77.47) (angle 90) (layer Edge.Cuts) (width 0.1))
+  (gr_line (start 170.815 64.135) (end 170.815 77.47) (angle 90) (layer Edge.Cuts) (width 0.1))
+  (gr_line (start 151.13 64.135) (end 170.815 64.135) (angle 90) (layer Edge.Cuts) (width 0.1))
+  (gr_line (start 151.13 53.34) (end 118.11 53.34) (angle 90) (layer Edge.Cuts) (width 0.1))
+  (gr_line (start 151.13 64.135) (end 151.13 53.34) (angle 90) (layer Edge.Cuts) (width 0.1))
   (gr_line (start 118.11 152.4) (end 187.96 152.4) (angle 90) (layer Edge.Cuts) (width 0.1))
-  (gr_line (start 118.11 53.34) (end 160.02 53.34) (angle 90) (layer Edge.Cuts) (width 0.1))
   (gr_line (start 118.11 53.34) (end 118.11 152.4) (angle 90) (layer Edge.Cuts) (width 0.1))
-  (gr_line (start 173.355 77.47) (end 158.115 77.47) (angle 90) (layer Edge.Cuts) (width 0.1))
   (gr_line (start 158.115 114.935) (end 158.115 77.47) (angle 90) (layer Edge.Cuts) (width 0.1))
   (gr_line (start 187.96 114.935) (end 158.115 114.935) (angle 90) (layer Edge.Cuts) (width 0.1))
